File: schematics/rp2040.kicad_sch (KiCad schematic)
At the start: 27 parts, among them SW1 TS-1088-AR02016, U1 RP2040, U2 W25Q128JVSIQTR, X1 X322512MSB4SI

Commit message: Organise capacitors
Connections:
- net GND: now also USB1.13 (SHELL), USB1.14 (SHELL)
Changed lines of the file:
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@@
 	)
 	(junction
+		(at 203.2 147.32)
+		(diameter 0)
+		(color 0 0 0 0)
+	)
+	(junction
 		(at 72.39 80.01)
 		(diameter 0)
@@
 	)
 	(junction
+		(at 254 142.24)
+		(diameter 0)
+		(color 0 0 0 0)
+	)
+	(junction
 		(at 222.25 81.28)
 		(diameter 0)
@@
 	(wire
 		(pts
+			(xy 203.2 147.32) (xy 203.2 149.86)
+		)
+		(stroke
+			(width 0)
+			(type default)
+		)
+	)
+	(wire
+		(pts
 			(xy 229.87 132.08) (xy 226.06 132.08)
 		)
@@
 	(wire
 		(pts
+			(xy 251.46 142.24) (xy 254 142.24)
+		)
+		(stroke
+			(width 0)
+			(type default)
+		)
+	)
+	(wire
+		(pts
 			(xy 110.49 58.42) (xy 116.84 58.42)
 		)
@@
 	(wire
 		(pts
+			(xy 254 114.3) (xy 254 142.24)
+		)
+		(stroke
+			(width 0)
+			(type default)
+		)
+	)
+	(wire
+		(pts
 			(xy 156.21 99.06) (xy 156.21 93.98)
 		)
@@
 	(wire
 		(pts
+			(xy 251.46 114.3) (xy 254 114.3)
+		)
+		(stroke
+			(width 0)
+			(type default)
+		)
+	)
+	(wire
+		(pts
 			(xy 110.49 50.8) (xy 116.84 50.8)
 		)
@@
 	(wire
 		(pts
-			(xy 203.2 142.24) (xy 203.2 144.78)
+			(xy 254 147.32) (xy 203.2 147.32)
+		)
+		(stroke
+			(width 0)
+			(type default)
+		)
+	)
+	(wire
+		(pts
+			(xy 203.2 142.24) (xy 203.2 147.32)
 		)
 		(stroke
@@
 	(wire
 		(pts
+			(xy 254 142.24) (xy 254 147.32)
+		)
+		(stroke
+			(width 0)
+			(type default)
+		)
+	)
+	(wire
+		(pts
 			(xy 72.39 80.01) (xy 74.93 80.01)
 		)
@@
 	(symbol
 		(lib_id "power:GND")
-		(at 203.2 144.78 0)
+		(at 203.2 149.86 0)
 		(unit 1)
 		(exclude_from_sim no)
@@
 		(fields_autoplaced yes)
 		(property "Reference" "#PWR013"
-			(at 203.2 151.13 0)
+			(at 203.2 156.21 0)
 			(effects
 				(font
@@
 		)
 		(property "Value" "GND"
-			(at 203.2 149.86 0)
+			(at 203.2 154.94 0)
 			(effects
 				(font
@@
 		)
 		(property "Footprint" ""
-			(at 203.2 144.78 0)
+			(at 203.2 149.86 0)
 			(effects
 				(font
@@
 		)
 		(property "Datasheet" ""
-			(at 203.2 144.78 0)
+			(at 203.2 149.86 0)
 			(effects
 				(font
@@
 		)
 		(property "Description" "Power symbol creates a global label with name \"GND\" , ground"
-			(at 203.2 144.78 0)
+			(at 203.2 149.86 0)
 			(effects
 				(font
