File: schematics/rp2040.kicad_sch (KiCad schematic)
At the start: 27 parts, among them SW1 TS-1088-AR02016, U1 RP2040, U2 W25Q128JVSIQTR, X1 X322512MSB4SI

Commit message: update schematics
Parts:
- added C29, C30: 100n, Capacitor_SMD:C_0603_1608Metric, symbol Device:C
- added D4, D5, D6: LED, LED_SMD:LED_0603_1608Metric, symbol Device:LED
- added R19: 1k, Resistor_SMD:R_0603_1608Metric, symbol Device:R
- added R20, R21, R22: 68R, Resistor_SMD:R_0603_1608Metric, symbol Device:R
- added SW2: TS-1088-AR02016, easyeda2kicad:SW-SMD_L3.9-W3.0-P4.45, symbol easyeda2kicad:TS-1088-AR02016
- added U11: AMS1117-3.3_C347222, easyeda2kicad:SOT-223-4_L6.5-W3.5-P2.30-LS7.0-BR, symbol easyeda2kicad:AMS1117-3.3_C347222
Connections:
- net GND: now also X1.2 (GND), X1.4 (GND), C29.2, C30.2, D4.1 (K), D5.1 (K), D6.1 (K), SW2.1, U11.1 (ADJ(GND))
- net GPIO6: now also R22.1
- net GPIO7: now also R21.1
- net QSPI_SS: now also R4.1, R5.2
- net 3.3V: now reaches C15.1, U2.8 (VCC)
- net 3.3V: now also C10.1, C11.1, C3.1, C4.1, C5.1, C6.1, C7.1, C8.1, C9.1, R5.1, U1.1 (IOVDD), U1.10 (IOVDD), U1.22 (IOVDD), U1.33 (IOVDD), U1.42 (IOVDD), U1.43 (ADC_AVDD), U1.44 (VREG_IN), U1.48 (USB_VDD), U1.49 (IOVDD), C29.1, R19.1, R20.1, U11.2 (VOUT(TAB)), U11.4 (TAB); no longer R4.1, R5.2
- net at USB1.4 (CC1): now also R6.2; no longer R7.2
- net at USB1.10 (CC2): now also R7.2; no longer R6.2
- net +1V1 renamed 1.1V
- removed net +3.3V: C10.1, C11.1, C3.1, C4.1, C5.1, C6.1, C7.1, C8.1, C9.1, R5.1, U1.1 (IOVDD), U1.10 (IOVDD), U1.22 (IOVDD), U1.26 (RUN), U1.33 (IOVDD), U1.42 (IOVDD), U1.43 (ADC_AVDD), U1.44 (VREG_IN), U1.48 (USB_VDD), U1.49 (IOVDD)
- net +5V renamed VBUS
- net VBUS: now also C30.1, U11.3 (VIN)
- new net: D6.2 (A), R22.2
- new net: D4.2 (A), R20.2
- new net: D5.2 (A), R21.2
- new net RUN: R19.2, SW2.2, U1.26 (RUN)
- no-connect marks 6 -> 4
Other:
- moved on the sheet: C10, C11, C12, C13, C14, C3, C4, C5, C6, C7, C8, C9
